Commit message: fixed camera mount on the urdf

File: interbotix_ws/install/interbotix_xslocobot_descriptions/share/interbotix_xslocobot_descriptions/urdf/camera_tower.urdf.xacro (robot description, xacro)
@@ -3,5 +3,6 @@
   <xacro:macro name="camera_tower" params="*origin *inertial">
     <joint name="camera_tower" type="fixed">
-      <xacro:insert_block name="origin"/>
+      <!--<xacro:insert_block name="origin"/> -->
+      <origin rpy="0 0 0" xyz="-0.03751 0 0.13775"/>
       <parent
         link="${robot_name}/base_link"/>
@@ -11,25 +12,26 @@
     <link name="${robot_name}/camera_tower_link">
       <visual>
-        <origin
-          rpy="0 0 0"
-          xyz="0 0 0"/>
+        <origin rpy="1.57079632679 0 1.57079632679" xyz="0.03751 0 -0.146150"/>
         <geometry>
           <mesh
-            filename="package://interbotix_xslocobot_descriptions/meshes/locobot_meshes/${base_type}_version/locobot_camera_tower_${camera_tower_size}.stl"
-            scale="${mesh_scale}"/>
+            filename="package://interbotix_xslocobot_descriptions/cmu_meshes/interbotix_cam_mount.stl" scale="0.001 0.001 0.001"/>
         </geometry>
-        <material name="interbotix_black"/>
+        <material name="">
+            <color rgba="0.792156862745098 0.819607843137255 0.933333333333333 1"/>
+        </material>
       </visual>
       <collision>
-        <origin
-          rpy="0 0 0"
-          xyz="0 0 0"/>
+        <origin rpy="1.57079632679 0 1.57079632679" xyz="0.03751 0 -0.146150"/>
         <geometry>
           <mesh
-            filename="package://interbotix_xslocobot_descriptions/meshes/locobot_meshes/${base_type}_version/locobot_camera_tower_${camera_tower_size}_simple.stl"
-            scale="${mesh_scale}"/>
+            filename="package://interbotix_xslocobot_descriptions/cmu_meshes/interbotix_cam_mount.stl" scale="0.001 0.001 0.001"/>
         </geometry>
       </collision>
-      <xacro:insert_block name="inertial"/>
+      <inertial>
+            <origin rpy="0 0 1.57079632679" xyz="-0.0053535000 -0.0030566200 0.1091990000"/>
+            <!-- <mass value="1"/> -->
+            <mass value="2.091937"/>
+            <inertia ixx="0.0376600000" ixy="-0.0001113000" ixz="-0.0004178000" iyy="0.0440300000" iyz="0.0001531000" izz="0.0116800000"/>
+        </inertial>
     </link>
     <gazebo reference="${robot_name}/camera_tower_link">

File: interbotix_ws/install/interbotix_xslocobot_descriptions/share/interbotix_xslocobot_descriptions/urdf/locobot.urdf.xacro (robot description, xacro)
@@ -91,4 +91,5 @@
     <xacro:if value="${arm_type == 'mobile_wx200'}">
       <xacro:if value="${base_type == 'kobuki'}">
+        <!--
         <xacro:arm_cradle>
           <origin
@@ -96,4 +97,5 @@
             xyz="0.0215 0 0.1195"/>
         </xacro:arm_cradle>
+        -->
       </xacro:if> <!-- base_type == 'kobuki' -->
       <xacro:if value="${base_type == 'create3'}">

File: interbotix_ws/install/interbotix_xslocobot_descriptions/share/interbotix_xslocobot_descriptions/urdf/pan_and_tilt.urdf.xacro (robot description, xacro)
@@ -9,5 +9,6 @@
         upper="${pi/2}"
         velocity="${pi}"/>
-      <xacro:insert_block name="origin"/>
+      <!--xacro:insert_block name="origin"/-->
+      <origin rpy="0 0 0" xyz="0.01755 -0.00008 0.3975"/>
       <parent
         link="${robot_name}/camera_tower_link"/>
@@ -21,36 +22,30 @@
       <visual>
         <origin
-          rpy="0 0 ${pi/2}"
-          xyz="0 0 0"/>
-        <geometry>
-          <mesh
-            filename="package://interbotix_xslocobot_descriptions/meshes/locobot_meshes/locobot_pan.stl"
-            scale="0.001 0.001 0.001"/>
-        </geometry>
-        <material name="interbotix_black"/>
+          rpy="0 0 0"
+          xyz="0 0 0"/> <!-- rpy= 0 0 ${pi/2}-->
+        <geometry>
+          <mesh
+            filename="package://interbotix_xslocobot_descriptions/cmu_meshes/tilt_link.stl"
+            scale="1 1 1"/> <!-- scale="0.001 0.001 0.001" -->
+        </geometry>
+        <material name="">
+          <color rgba="0.250980392156863 0.250980392156863 0.250980392156863 1"/>
+        </material>
       </visual>
       <collision>
         <origin
-          rpy="0 0 ${pi/2}"
-          xyz="0 0 0"/>
-        <geometry>
-          <mesh
-            filename="package://interbotix_xslocobot_descriptions/meshes/locobot_meshes/locobot_pan.stl"
-            scale="0.001 0.001 0.001"/>
+          rpy="0 0 0"
+          xyz="0 0 0"/>
+        <geometry>
+          <mesh
+            filename="package://interbotix_xslocobot_descriptions/cmu_meshes/tilt_link.stl"
+            scale="1 1 1"/> <!-- scale="0.001 0.001 0.001" -->
         </geometry>
       </collision>
       <inertial>
-        <origin
-          rpy="0 0 ${pi/2}"
-          xyz="0.012 0.000496 0.018504"/>
-        <mass value="0.098997"/>
-        <inertia
-          ixx="0.0000276300"
-          ixy="0.0000000418"
-          ixz="0.0000005145"
-          iyy="0.0000204300"
-          iyz="-0.0000000421"
-          izz="0.0000276300"/>
-      </inertial>
+            <origin rpy="0 0 0" xyz="-1.35308431126191E-16 -2.97071395261028E-17 0.0220876265081744"/>
+            <mass value="0.0182769203076134"/>
+            <inertia ixx="1.32243845065555E-05" ixy="5.07660179129181E-13" ixz="1.067515220067E-20" iyy="7.13386116649085E-06" iyz="-1.32882457845217E-20" izz="7.83291781352837E-06"/>
+        </inertial>
     </link>
     <gazebo reference="${robot_name}/pan_link">
@@ -61,11 +56,11 @@
       <axis xyz="0 1 0"/>
       <limit
-        effort="2"
-        lower="${-pi/2}"
-        upper="${radians(75)}"
-        velocity="${pi}"/>
+        effort="1"
+        lower="-1.57"
+        upper="1.57"
+        velocity="1"/>
       <origin
         rpy="0 0 0"
-        xyz="0.025034 0 0.019"/>
+        xyz="0.0 0 0.05"/>
       <parent
         link="${robot_name}/pan_link"/>
@@ -100,36 +95,30 @@
       <visual>
         <origin
-          rpy="0 0 ${pi/2}"
-          xyz="0 0 0"/>
-        <geometry>
-          <mesh
-            filename="package://interbotix_xslocobot_descriptions/meshes/locobot_meshes/locobot_tilt.stl"
-            scale="0.001 0.001 0.001"/>
-        </geometry>
-        <material name="interbotix_black"/>
+          rpy="0 0 0"
+          xyz="0 0 0"/>
+        <geometry>
+          <mesh
+            filename="package://interbotix_xslocobot_descriptions/cmu_meshes/roll_link.stl"
+            scale="1 1 1"/>
+        </geometry>
+        <material name="">
+            <color rgba="0.792156862745098 0.819607843137255 0.933333333333333 1"/>
+        </material>
       </visual>
       <collision>
         <origin
-          rpy="0 0 ${pi/2}"
-          xyz="0 0 0"/>
-        <geometry>
-          <mesh
-            filename="package://interbotix_xslocobot_descriptions/meshes/locobot_meshes/locobot_tilt.stl"
-            scale="0.001 0.001 0.001"/>
+          rpy="0 0 0"
+          xyz="0 0 0"/>
+        <geometry>
+          <mesh
+            filename="package://interbotix_xslocobot_descriptions/cmu_meshes/roll_link.stl"
+            scale="1 1 1"/>
         </geometry>
       </collision>
       <inertial>
-        <origin
-          rpy="0 0 ${pi/2}"
-          xyz="0.0237737000 -0.0000016331 0.0000077432"/>
-        <mass value="0.019845"/>
-        <inertia
-          ixx="0.0000021677"
-          ixy="0.0000000000"
-          ixz="0.0000000001"
-          iyy="0.0000063634"
-          iyz="0.0000000003"
-          izz="0.0000066157"/>
-      </inertial>
+            <origin rpy="0 0 0" xyz="0.0168744200088311 -0.000442984145897884 -0.00405256422002387"/>
+            <mass value="0.0547677687275323"/>
+            <inertia ixx="1.07071738005716E-05" ixy="-1.46854788384565E-07" ixz="5.59529059364376E-08" iyy="1.77011620295824E-05" iyz="1.27587154712834E-09" izz="2.01583693170578E-05"/>
+        </inertial>
     </link>
     <gazebo reference="${robot_name}/tilt_link">
@@ -137,8 +126,9 @@
       <self_collide>true</self_collide>
     </gazebo>
+    <!-- Camera Model -->
     <joint name="camera" type="fixed">
       <origin
         rpy="0 0 0"
-        xyz="0.05318 0.0175 0.000009"/>
+        xyz="0.06705 0.0 -0.00425"/>
       <parent
         link="${robot_name}/tilt_link"/>
@@ -156,10 +146,9 @@
         <geometry>
           <mesh
-            filename="package://interbotix_xslocobot_descriptions/meshes/locobot_meshes/locobot_camera.stl"
-            scale="0.001 0.001 0.001"/>
+            filename="package://interbotix_xslocobot_descriptions/cmu_meshes/camera_link.stl"
+            scale="1 1 1"/>
         </geometry>
         <material name="">
-          <color
-            rgba="0.55 0.55 0.55 1"/>
+          <color rgba="0.792156862745098 0.819607843137255 0.933333333333333 1"/>
         </material>
       </visual>
@@ -170,21 +159,13 @@
         <geometry>
           <mesh
-            filename="package://interbotix_xslocobot_descriptions/meshes/locobot_meshes/locobot_camera.stl"
-            scale="0.001 0.001 0.001"/>
+            filename="package://interbotix_xslocobot_descriptions/cmu_meshes/camera_link.stl"
+            scale="1 1 1"/>
         </geometry>
       </collision>
       <inertial>
-        <origin
-          rpy="0 0 0"
-          xyz="-0.008972 -0.015818 0.000003"/>
-        <mass value="0.072"/>
-        <inertia
-          ixx="0.0000465400"
-          ixy="0.0000003028"
-          ixz="0.0000000245"
-          iyy="0.0000069128"
-          iyz="0.0000000248"
-          izz="0.0000468600"/>
-      </inertial>
+            <origin rpy="0 0 0" xyz="-0.0132722976093535 0.00168171470080143 2.49829664994428E-06"/>
+            <mass value="0.0381925651163644"/>
+            <inertia ixx="2.4688255642946E-05" ixy="1.60697655569215E-07" ixz="1.2993241737711E-08" iyy="3.66669176935806E-06" iyz="1.30215657011203E-08" izz="2.48602467766615E-05"/>
+        </inertial>
     </link>
     <gazebo reference="camera_${robot_name}_link">
