Commit message: found the error was the fingers

File: interbotix_ws/install/interbotix_xslocobot_descriptions/share/interbotix_xslocobot_descriptions/urdf/arms/mobile_wx200.urdf.xacro (robot description, xacro)
@@ -42,5 +42,5 @@
       <geometry>
         <mesh
-          filename="${mesh_directory}/base.stl"
+          filename="package://interbotix_xslocobot_descriptions/cmu_meshes/mobile_base.STL"
           scale="0.001 0.001 0.001"/>
       </geometry>
@@ -53,5 +53,5 @@
       <geometry>
         <mesh
-          filename="${mesh_directory}/base.stl"
+          filename="package://interbotix_xslocobot_descriptions/cmu_meshes/mobile_base.STL"
           scale="0.001 0.001 0.001"/>
       </geometry>
@@ -80,5 +80,5 @@
     <origin
       rpy="0 0 0"
-      xyz="0 0 0.066175"/>
+      xyz="0 0 0.0655"/>
     <parent
       link="${robot_name}/arm_base_link"/>
@@ -92,10 +92,9 @@
     <visual>
       <origin
-        rpy="0 0 ${pi/2}"
-        xyz="0 0 -0.003"/>
-      <geometry>
-        <mesh
-          filename="${mesh_directory}/shoulder.stl"
-          scale="0.001 0.001 0.001"/>
+        rpy="0 0 0"
+        xyz="0 0 -0.000"/>
+      <geometry>
+        <mesh
+          filename="package://interbotix_xslocobot_descriptions/cmu_meshes/shoulder_link.STL"/>
       </geometry>
       <material name="interbotix_black"/>
@@ -103,10 +102,10 @@
     <collision>
       <origin
-        rpy="0 0 ${pi/2}"
-        xyz="0 0 -0.003"/>
-      <geometry>
-        <mesh
-          filename="${mesh_directory}/shoulder.stl"
-          scale="0.001 0.001 0.001"/>
+        rpy="0 0 0"
+        xyz="0 0 -0.000"/>
+      <geometry>
+        <mesh
+          filename="package://interbotix_xslocobot_descriptions/cmu_meshes/shoulder_link.STL"
+          />
       </geometry>
     </collision>
@@ -511,5 +510,5 @@
               <mesh
                 filename="${mesh_directory}/gripper_finger.stl"
-                scale="0.001 0.001 0.001"/>
+                />
             </geometry>
             <material name="interbotix_black"/>
@@ -522,5 +521,5 @@
               <mesh
                 filename="${mesh_directory}/gripper_finger.stl"
-                scale="0.001 0.001 0.001"/>
+                />
             </geometry>
           </collision>

File: interbotix_ws/src/interbotix_ros_rovers/interbotix_ros_xslocobots/interbotix_xslocobot_descriptions/urdf/arms/mobile_wx200.urdf.xacro (robot description, xacro)
@@ -42,5 +42,5 @@
       <geometry>
         <mesh
-          filename="${mesh_directory}/base.stl"
+          filename="package://interbotix_xslocobot_descriptions/cmu_meshes/mobile_base.STL"
           scale="0.001 0.001 0.001"/>
       </geometry>
@@ -53,5 +53,5 @@
       <geometry>
         <mesh
-          filename="${mesh_directory}/base.stl"
+          filename="package://interbotix_xslocobot_descriptions/cmu_meshes/mobile_base.STL"
           scale="0.001 0.001 0.001"/>
       </geometry>
@@ -80,5 +80,5 @@
     <origin
       rpy="0 0 0"
-      xyz="0 0 0.066175"/>
+      xyz="0 0 0.0655"/>
     <parent
       link="${robot_name}/arm_base_link"/>
@@ -92,10 +92,9 @@
     <visual>
       <origin
-        rpy="0 0 ${pi/2}"
-        xyz="0 0 -0.003"/>
-      <geometry>
-        <mesh
-          filename="${mesh_directory}/shoulder.stl"
-          scale="0.001 0.001 0.001"/>
+        rpy="0 0 0"
+        xyz="0 0 -0.000"/>
+      <geometry>
+        <mesh
+          filename="package://interbotix_xslocobot_descriptions/cmu_meshes/shoulder_link.STL"/>
       </geometry>
       <material name="interbotix_black"/>
@@ -103,10 +102,10 @@
     <collision>
       <origin
-        rpy="0 0 ${pi/2}"
-        xyz="0 0 -0.003"/>
-      <geometry>
-        <mesh
-          filename="${mesh_directory}/shoulder.stl"
-          scale="0.001 0.001 0.001"/>
+        rpy="0 0 0"
+        xyz="0 0 -0.000"/>
+      <geometry>
+        <mesh
+          filename="package://interbotix_xslocobot_descriptions/cmu_meshes/shoulder_link.STL"
+          />
       </geometry>
     </collision>
